Commit message: 20241121

File: src/sipder_robot/xacro/plugin.xacro (robot description, xacro)
@@ -11,5 +11,5 @@
         <plugin name="p3d_base_controller" filename="libgazebo_ros_p3d.so">
             <alwaysOn>true</alwaysOn>
-            <updateRate>50.0</updateRate>
+            <updateRate>100.0</updateRate>
             <bodyName>base_link</bodyName>            <!-- 替换为你的基坐标系名称 -->
             <topicName>/Odometry</topicName>            <!-- 自定义的话题名称 -->
@@ -20,6 +20,3 @@
         </plugin>
     </gazebo>
-    <plugin name="triangle_draw_plugin" filename="libTriangleDrawPlugin.so">
-        <topicName>/triangle_Point</topicName>
-    </plugin>
 </robot>

File: src/sipder_robot/xacro/root_.xacro (robot description, xacro)
@@ -1,5 +1,5 @@
 <?xml version="1.0"?>
 <robot xmlns:xacro="http://www.ros.org/wiki/xacro" name="base_traj">
- <link name="world" />
+  <link name="world" />
   <joint name="world_joint" type="fixed">
     <parent link="world" />
@@ -20,5 +20,5 @@
     </inertial>
   </link>
-    <!--Note that the "topicName" is the topic name in launch file, it should be the same.
+  <!--Note that the "topicName" is the topic name in launch file, it should be the same.
 	Here, topicName is "Odometry" and so do it in the libgazebo_ros_p3d-->
   <gazebo reference="root">
@@ -29,3 +29,10 @@
     </visual>
   </gazebo>
+  <gazebo reference="root">
+    <visual>
+      <plugin filename="libdraw_triangle.so" name="drawtrianglePlugin">
+        <topicName>/triangle_points</topicName>
+      </plugin>
+    </visual>
+  </gazebo>
 </robot>
