Commit message: 20241122

File: src/sipder_robot/urdf/sipder_robot.urdf (robot description, URDF)
Before this commit: robot sipder_robot, 20 links, 19 joints
Joints:
- joint shank2foot1: type fixed -> revolute
- joint shank2foot2: type fixed -> revolute
- joint shank2foot4: type fixed -> revolute

File: src/sipder_robot/xacro/gazebo/foot_suction_cups.xacro (robot description, xacro)
@@ -27,14 +27,4 @@
         <dynamics damping="0.0" friction="10"/>
     </joint>
-    <gazebo>
-        <plugin name="gazebo_ros_vacuum_gripper" filename="libgazebo_ros_vacuum_gripper.so">
-            <robotNamespace>/spibot_vacuum_gripper1</robotNamespace>
-            <bodyName>vacuum_gripper1</bodyName>
-            <topicName>BR_suction_state</topicName>
-            <maxForce>400</maxForce>
-            <maxDistance>5.05</maxDistance>
-            <minDistance>0.01</minDistance>
-        </plugin>
-    </gazebo>
     <gazebo reference="vacuum_gripper1">
         <mu1>50</mu1>
@@ -71,14 +61,4 @@
         <dynamics damping="0.0" friction="10"/>
     </joint>
-    <gazebo>
-        <plugin name="gazebo_ros_vacuum_gripper" filename="libgazebo_ros_vacuum_gripper.so">
-            <robotNamespace>/spibot_vacuum_gripper2</robotNamespace>
-            <bodyName>vacuum_gripper2</bodyName>
-            <topicName>FR_suction_state</topicName>
-            <maxForce>400</maxForce>
-            <maxDistance>5.05</maxDistance>
-            <minDistance>0.01</minDistance>
-        </plugin>
-    </gazebo>
     <gazebo reference="vacuum_gripper2">
         <mu1>50</mu1>
@@ -115,14 +95,4 @@
         <dynamics damping="0.0" friction="10"/>
     </joint>
-    <gazebo>
-        <plugin name="gazebo_ros_vacuum_gripper" filename="libgazebo_ros_vacuum_gripper.so">
-            <robotNamespace>/spibot_vacuum_gripper3</robotNamespace>
-            <bodyName>vacuum_gripper3</bodyName>
-            <topicName>FL_suction_state</topicName>
-            <maxForce>400</maxForce>
-            <maxDistance>5.05</maxDistance>
-            <minDistance>0.01</minDistance>
-        </plugin>
-    </gazebo>
     <gazebo reference="vacuum_gripper3">
         <mu1>50</mu1>
@@ -159,14 +129,4 @@
         <dynamics damping="0.0" friction="10"/>
     </joint>
-    <gazebo>
-        <plugin name="gazebo_ros_vacuum_gripper" filename="libgazebo_ros_vacuum_gripper.so">
-            <robotNamespace>/spibot_vacuum_gripper4</robotNamespace>
-            <bodyName>vacuum_gripper4</bodyName>
-            <topicName>BL_suction_state</topicName>
-            <maxForce>400</maxForce>
-            <maxDistance>5.05</maxDistance>
-            <minDistance>0.01</minDistance>
-        </plugin>
-    </gazebo>
     <gazebo reference="vacuum_gripper4">
         <mu1>50</mu1>

File: src/sipder_robot/xacro/root_.xacro (robot description, xacro)
@@ -32,5 +32,5 @@
     <visual>
       <plugin filename="libdraw_triangle.so" name="drawtrianglePlugin">
-        <topicName>/triangle_points</topicName>
+        <topicName>/spibot_gazebo/draw/triangle_points</topicName>
       </plugin>
     </visual>

File: src/sipder_robot/xacro/spibot.xacro (robot description, xacro)
@@ -547,56 +547,37 @@
         </collision>
     </link>
-    <joint name="shank2foot1" type="fixed">
+    <!-- type="revolute" : 发布连杆关系的话题就是在/tf -->
+    <!-- type="fixed" : 发布连杆关系的话题就是在/tf_static -->
+    <joint name="shank2foot1" type="revolute">
         <origin xyz="0.36572 0 0.00075" rpy="-1.5818 -1.5708 -1.5598" />
         <parent link="shank1" />
         <child link="foot1" />
         <axis xyz="0 0 -1" />
-    </joint>
-    <joint name="shank2foot2" type="fixed">
+        <limit effort="50" velocity="50" lower="0" upper="0" />
+        <dynamics damping="0.0" friction="10"/>
+    </joint>
+    <joint name="shank2foot2" type="revolute">
         <origin xyz="0.36572 0 0.00075" rpy="-1.5718 -1.5708 -1.5698" />
         <parent link="shank2" />
         <child link="foot2" />
         <axis xyz="0 0 -1" />
-    </joint>
-    <joint name="shank2foot3" type="fixed">
+        <limit effort="50" velocity="50" lower="0" upper="0" />
+        <dynamics damping="0.0" friction="10"/>
+    </joint>
+    <joint name="shank2foot3" type="revolute">
         <origin xyz="0.36572 0 0.00075" rpy="0 1.5708 0" />
         <parent link="shank3" />
         <child link="foot3" />
         <axis xyz="0 0 -1" />
-    </joint>
-    <joint name="shank2foot4" type="fixed">
+        <limit effort="50" velocity="50" lower="0" upper="0" />
+        <dynamics damping="0.0" friction="10"/>
+    </joint>
+    <joint name="shank2foot4" type="revolute">
         <origin xyz="0.36572 0 0.00075" rpy="0 1.5708 0" />
         <parent link="shank4" />
         <child link="foot4" />
         <axis xyz="0 0 -1" />
-    </joint>
-    <!-- 定义球铰链关节 -->
-    <!-- <joint name="shank2foot1" type="revolute">
-        <origin xyz="0.36572 0 0.00075" rpy="-1.5818 -1.5708 -1.5598"/>
-        <parent link="shank1"/>
-        <child link="foot1"/>
-        <axis xyz="0 0 0"/>
-        <limit lower="-3.14" upper="3.14" effort="500" velocity="40" />
-    </joint>
-    <joint name="shank2foot2" type="revolute">
-        <origin xyz="0.36572 0 0.00075" rpy="-1.5718 -1.5708 -1.5698"/>
-        <parent link="shank2"/>
-        <child link="foot2"/>
-        <axis xyz="0 0 0"/>
-        <limit lower="-3.14" upper="3.14" effort="500" velocity="40" />
-    </joint>
-    <joint name="shank2foot3" type="revolute">
-        <origin xyz="0.36572 0 0.00075" rpy="0 1.5708 0"/>
-        <parent link="shank3"/>
-        <child link="foot3"/>
-        <axis xyz="0 0 0"/>
-        <limit lower="-3.14" upper="3.14" effort="500" velocity="40" />
-    </joint>
-    <joint name="shank2foot4" type="revolute">
-        <origin xyz="0.36572 0 0.00075" rpy="0 1.5708 0"/>
-        <parent link="shank4"/>
-        <child link="foot4"/>
-        <axis xyz="0 0 0"/>
-        <limit lower="-3.14" upper="3.14" effort="500" velocity="40" />
-    </joint> -->
+        <limit effort="50" velocity="50" lower="0" upper="0" />
+        <dynamics damping="0.0" friction="10"/>
+    </joint>
 </robot>
