Commit message: 20241211

File: src/sipder_robot/urdf/SpibotRl.urdf (robot description, URDF)
Before this commit: robot SpibotRl, 34 links, 33 joints
Links:
- link FL_calf: geometry visual mesh filename=../meshes/FL_calf.STL
- link FL_foot: geometry visual mesh filename=../meshes/FL_foot.STL
- link FL_hip: geometry visual mesh filename=../meshes/FL_hip.STL
- link FL_thigh: geometry visual mesh filename=../meshes/FL_thigh.STL
- link FR_calf: geometry visual mesh filename=../meshes/FR_calf.STL
- link FR_foot: geometry visual mesh filename=../meshes/FR_foot.STL
- link FR_hip: geometry visual mesh filename=../meshes/FR_hip.STL
- link FR_thigh: geometry visual mesh filename=../meshes/FR_thigh.STL
- link RL_calf: geometry visual mesh filename=../meshes/RL_calf.STL
- link RL_foot: geometry visual mesh filename=../meshes/RL_foot.STL
- link RL_hip: geometry visual mesh filename=../meshes/RL_hip.STL
- link RL_thigh: geometry visual mesh filename=../meshes/RL_thigh.STL
- link RR_calf: geometry visual mesh filename=../meshes/RR_calf.STL
- link RR_foot: geometry visual mesh filename=../meshes/RR_foot.STL
- link RR_hip: geometry visual mesh filename=../meshes/RR_hip.STL
- link RR_thigh: geometry visual mesh filename=../meshes/RR_thigh.STL
- link base: geometry collision box size=0.304 0.304 0.109; visual mesh filename=../meshes/base.STL
- link imu: geometry visual mesh filename=../meshes/imu.STL

File: src/sipder_robot/xacro/const.xacro (robot description, xacro)
@@ -5,5 +5,5 @@
     <xacro:property name="base_com_y" value="-0.0053069"/>
     <xacro:property name="base_com_z" value="0.074681"/>
-    <xacro:property name="base_mass" value="2.8003"/>
+    <xacro:property name="base_mass" value="8.956765"/>
     <xacro:property name="base_ixx" value="0.0051964"/>
     <xacro:property name="base_ixy" value="1.4763E-06"/>

Commit message: 20241223

File: src/sipder_robot/urdf/SpibotRl.urdf (robot description, URDF)
Before this commit: robot SpibotRl, 34 links, 33 joints
Links:
- removed link FL_foot_col
- removed link FR_foot_col
- removed link RL_foot_col
- removed link RR_foot_col
- removed link imu
- added link base_inertia, mass 8.956765
- added link imu_col; collision box size=0.025 0.09 0.025
- added link imu_link, mass 0.01; visual mesh filename=../meshes/imu.STL
- link FL_foot: geometry collision box size=0.108 0.108 0.108; visual mesh filename=../meshes/FL_foot.STL
- link FR_foot: geometry collision box size=0.108 0.108 0.108; visual mesh filename=../meshes/FR_foot.STL
- link RL_foot: geometry collision box size=0.108 0.108 0.108; visual mesh filename=../meshes/RL_foot.STL
- link RR_foot: geometry collision box size=0.108 0.108 0.108; visual mesh filename=../meshes/RR_foot.STL
- link base: mass 8.956765 -> None
Joints:
- removed joint FL_foot_col_joint
- removed joint FR_foot_col_joint
- removed joint RL_foot_col_joint
- removed joint RR_foot_col_joint
- added joint base_to_base_inertia: type fixed, parent base, child base_inertia, origin xyz=0 0 0 rpy=0 0 0
- added joint imu_col_joint: type fixed, parent imu_link, child imu_col, origin xyz=-0.0125 0 0 rpy=0 0 0, axis 0 -1 0, limit lower=-2.0 upper=1.0 effort=100 velocity=30
- joint RL_thigh_joint: limit lower=-2.0 upper=1.0 effort=100 velocity=30 -> lower=-1.0 upper=2.0 effort=100 velocity=30
- joint imu_joint: axis 0 0 0 -> (none); child imu -> imu_link

File: src/sipder_robot/xacro/gazebo/foot_add_grippers.xacro (robot description, xacro)
@@ -7,5 +7,5 @@
             <origin rpy="0 0 0" xyz="0 0 0"/>
             <geometry>
-                <cylinder radius="0.05" length="0.01"/>
+                <cylinder length="0.005" radius="0.05" />
             </geometry>
             <material name="transparent">
@@ -23,5 +23,5 @@
         <parent link="foot1" />
         <child link="vacuum_gripper1" />
-        <origin rpy="0 0 0" xyz="0 0 0.052" />
+        <origin rpy="0 0 0" xyz="0 0 0" />
         <limit effort="50" velocity="50" lower="0" upper="0" />
         <dynamics damping="0.0" friction="10"/>
@@ -41,5 +41,5 @@
             <origin rpy="0 0 0" xyz="0 0 0"/>
             <geometry>
-                <cylinder radius="0.05" length="0.01"/>
+                <cylinder length="0.005" radius="0.05" />
             </geometry>
             <material name="transparent">
@@ -57,5 +57,5 @@
         <parent link="foot2" />
         <child link="vacuum_gripper2" />
-        <origin rpy="0 0 0" xyz="0 0 0.052" />
+        <origin rpy="0 0 0" xyz="0 0 0" />
         <limit effort="50" velocity="50" lower="0" upper="0" />
         <dynamics damping="0.0" friction="10"/>
@@ -75,5 +75,5 @@
             <origin rpy="0 0 0" xyz="0 0 0"/>
             <geometry>
-                <cylinder radius="0.05" length="0.01"/>
+                <cylinder length="0.005" radius="0.05" />
             </geometry>
             <material name="transparent">
@@ -91,5 +91,5 @@
         <parent link="foot3" />
         <child link="vacuum_gripper3" />
-        <origin rpy="0 0 0" xyz="0 0 0.052" />
+        <origin rpy="0 0 0" xyz="0 0 0" />
         <limit effort="50" velocity="50" lower="0" upper="0" />
         <dynamics damping="0.0" friction="10"/>
@@ -109,5 +109,5 @@
             <origin rpy="0 0 0" xyz="0 0 0"/>
             <geometry>
-                <cylinder radius="0.05" length="0.01"/>
+                <cylinder length="0.005" radius="0.05" />
             </geometry>
             <material name="transparent">
@@ -125,5 +125,5 @@
         <parent link="foot4" />
         <child link="vacuum_gripper4" />
-        <origin rpy="0 0 0" xyz="0 0 0.052" />
+        <origin rpy="0 0 0" xyz="0 0 0" />
         <limit effort="50" velocity="50" lower="0" upper="0" />
         <dynamics damping="0.0" friction="10"/>

File: src/sipder_robot/xacro/spibot_with_sensors.xacro (robot description, xacro)
@@ -2,5 +2,5 @@
 <robot name="spibot_with_sensors"
     xmlns:xacro="http://www.ros.org/wiki/xacro">
-    <xacro:include filename="spibot.xacro"/>
+    <xacro:include filename="spibot_new.xacro"/>
     <!-- 集成运动控制 -->
     <!-- 给机器人的camera增加深度相机以生成深度图像 -->
