Commit message: 20241210

File: src/sipder_robot/urdf/WindTurbine_Blade.urdf (robot description, URDF)
Before this commit: robot WindTurbine_Blade, 1 links, 0 joints
Links:
- link base_link: geometry collision mesh filename=package://sipder_robot/meshes/spibot/WindTurbine_Blade.STL; visual mesh filename=package://sipder_robot/meshes/spibot/WindTurbine_Blade.STL

File: src/sipder_robot/urdf/sipder_robot.urdf (robot description, URDF)
Before this commit: robot sipder_robot, 20 links, 19 joints
Links:
- link base_link: geometry collision mesh filename=package://sipder_robot/meshes/spibot/base_link.STL; visual mesh filename=package://sipder_robot/meshes/spibot/base_link.STL
- link camera: geometry collision mesh filename=package://sipder_robot/meshes/spibot/camera.STL; visual mesh filename=package://sipder_robot/meshes/spibot/camera.STL
- link foot1: geometry collision mesh filename=package://sipder_robot/meshes/spibot/foot1.STL; visual mesh filename=package://sipder_robot/meshes/spibot/foot1.STL
- link foot2: geometry collision mesh filename=package://sipder_robot/meshes/spibot/foot2.STL; visual mesh filename=package://sipder_robot/meshes/spibot/foot2.STL
- link foot3: geometry collision mesh filename=package://sipder_robot/meshes/spibot/foot3.STL; visual mesh filename=package://sipder_robot/meshes/spibot/foot3.STL
- link foot4: geometry collision mesh filename=package://sipder_robot/meshes/spibot/foot4.STL; visual mesh filename=package://sipder_robot/meshes/spibot/foot4.STL
- link hip1: geometry collision mesh filename=package://sipder_robot/meshes/spibot/hip1.STL; visual mesh filename=package://sipder_robot/meshes/spibot/hip1.STL
- link hip2: geometry collision mesh filename=package://sipder_robot/meshes/spibot/hip2.STL; visual mesh filename=package://sipder_robot/meshes/spibot/hip2.STL
- link hip3: geometry collision mesh filename=package://sipder_robot/meshes/spibot/hip3.STL; visual mesh filename=package://sipder_robot/meshes/spibot/hip3.STL
- link hip4: geometry collision mesh filename=package://sipder_robot/meshes/spibot/hip4.STL; visual mesh filename=package://sipder_robot/meshes/spibot/hip4.STL
- link lidar: geometry collision mesh filename=package://sipder_robot/meshes/spibot/lidar.STL; visual mesh filename=package://sipder_robot/meshes/spibot/lidar.STL
- link shank1: geometry collision mesh filename=package://sipder_robot/meshes/spibot/shank1.STL; visual mesh filename=package://sipder_robot/meshes/spibot/shank1.STL
- link shank2: geometry collision mesh filename=package://sipder_robot/meshes/spibot/shank2.STL; visual mesh filename=package://sipder_robot/meshes/spibot/shank2.STL
- link shank3: geometry collision mesh filename=package://sipder_robot/meshes/spibot/shank3.STL; visual mesh filename=package://sipder_robot/meshes/spibot/shank3.STL
- link shank4: geometry collision mesh filename=package://sipder_robot/meshes/spibot/shank4.STL; visual mesh filename=package://sipder_robot/meshes/spibot/shank4.STL
- link thigh1: geometry collision mesh filename=package://sipder_robot/meshes/spibot/thigh1.STL; visual mesh filename=package://sipder_robot/meshes/spibot/thigh1.STL
- link thigh2: geometry collision mesh filename=package://sipder_robot/meshes/spibot/thigh2.STL; visual mesh filename=package://sipder_robot/meshes/spibot/thigh2.STL
- link thigh3: geometry collision mesh filename=package://sipder_robot/meshes/spibot/thigh3.STL; visual mesh filename=package://sipder_robot/meshes/spibot/thigh3.STL
- link thigh4: geometry collision mesh filename=package://sipder_robot/meshes/spibot/thigh4.STL; visual mesh filename=package://sipder_robot/meshes/spibot/thigh4.STL

File: src/sipder_robot/xacro/spibot.xacro (robot description, xacro)
@@ -42,5 +42,5 @@
             <origin xyz="0 0 0" rpy="0 0 0" />
             <geometry>
-                <mesh filename="package://sipder_robot/meshes/base_link.STL" />
+                <mesh filename="package://sipder_robot/meshes/spibot/base_link.STL" />
             </geometry>
             <material name="White">
@@ -51,5 +51,5 @@
             <origin xyz="0 0 0" rpy="0 0 0" />
             <geometry>
-                <mesh filename="package://sipder_robot/meshes/base_link.STL" />
+                <box size="0.304 0.304 0.109" />
             </geometry>
         </collision>
@@ -63,5 +63,5 @@
             <origin xyz="0 0 0" rpy="0 0 0" />
             <geometry>
-                <mesh filename="package://sipder_robot/meshes/camera.STL" />
+                <mesh filename="package://sipder_robot/meshes/spibot/camera.STL" />
             </geometry>
             <material name="DarkGrey">
@@ -69,10 +69,4 @@
             </material>
         </visual>
-        <collision>
-            <origin xyz="0 0 0" rpy="0 0 0" />
-            <geometry>
-                <mesh filename="package://sipder_robot/meshes/camera.STL" />
-            </geometry>
-        </collision>
     </link>
     <joint name="base2camera" type="fixed">
@@ -82,13 +76,8 @@
     </joint>
     <link name="lidar">
-        <inertial>
-            <origin xyz="${lidar_com_x} ${lidar_com_y} ${lidar_com_z}" rpy="0 0 0" />
-            <mass value="${lidar_mass}" />
-            <inertia ixx="${lidar_ixx}" ixy="${lidar_ixy}" ixz="${lidar_ixz}" iyy="${lidar_iyy}" iyz="${lidar_iyz}" izz="${lidar_izz}" />
-        </inertial>
-        <visual>
-            <origin xyz="0 0 0" rpy="0 0 0" />
-            <geometry>
-                <mesh filename="package://sipder_robot/meshes/lidar.STL" />
+        <visual>
+            <origin xyz="0 0 0" rpy="0 0 0" />
+            <geometry>
+                <mesh filename="package://sipder_robot/meshes/spibot/lidar.STL" />
             </geometry>
             <material name="DarkSlateBlue">
@@ -96,10 +85,4 @@
             </material>
         </visual>
-        <collision>
-            <origin xyz="0 0 0" rpy="0 0 0" />
-            <geometry>
-                <mesh filename="package://sipder_robot/meshes/lidar.STL" />
-            </geometry>
-        </collision>
     </link>
     <joint name="base2lidar" type="fixed">
@@ -119,5 +102,5 @@
             <origin xyz="0 0 0" rpy="0 0 0" />
             <geometry>
-                <mesh filename="package://sipder_robot/meshes/hip1.STL" />
+                <mesh filename="package://sipder_robot/meshes/spibot/hip1.STL" />
             </geometry>
             <material name="IndianRed">
@@ -128,5 +111,5 @@
             <origin xyz="0 0 0" rpy="0 0 0" />
             <geometry>
-                <mesh filename="package://sipder_robot/meshes/hip1.STL" />
+                <mesh filename="package://sipder_robot/meshes/spibot/hip1.STL" />
             </geometry>
         </collision>
@@ -148,5 +131,5 @@
             <origin xyz="0 0 0" rpy="0 0 0" />
             <geometry>
-                <mesh filename="package://sipder_robot/meshes/thigh1.STL" />
+                <mesh filename="package://sipder_robot/meshes/spibot/thigh1.STL" />
             </geometry>
             <material name="Green">
@@ -157,5 +140,5 @@
             <origin xyz="0 0 0" rpy="0 0 0" />
             <geometry>
-                <mesh filename="package://sipder_robot/meshes/thigh1.STL" />
+                <mesh filename="package://sipder_robot/meshes/spibot/thigh1.STL" />
             </geometry>
         </collision>
@@ -177,5 +160,5 @@
             <origin xyz="0 0 0" rpy="0 0 0" />
             <geometry>
-                <mesh filename="package://sipder_robot/meshes/shank1.STL" />
+                <mesh filename="package://sipder_robot/meshes/spibot/shank1.STL" />
             </geometry>
             <material name="Cyan">
@@ -186,5 +169,5 @@
             <origin xyz="0 0 0" rpy="0 0 0" />
             <geometry>
-                <mesh filename="package://sipder_robot/meshes/shank1.STL" />
+                <mesh filename="package://sipder_robot/meshes/spibot/shank1.STL" />
             </geometry>
         </collision>
@@ -229,5 +212,5 @@
             <origin xyz="0 0 0" rpy="0 0 0" />
             <geometry>
-                <mesh filename="package://sipder_robot/meshes/foot1.STL" />
+                <mesh filename="package://sipder_robot/meshes/spibot/foot1.STL" />
             </geometry>
             <material name="SkyBlue">
@@ -238,5 +221,5 @@
             <origin xyz="0 0 0" rpy="0 0 0" />
             <geometry>
-                <mesh filename="package://sipder_robot/meshes/foot1.STL" />
+                <mesh filename="package://sipder_robot/meshes/spibot/foot1.STL" />
             </geometry>
         </collision>
@@ -252,5 +235,5 @@
             <origin xyz="0 0 0" rpy="0 0 0" />
             <geometry>
-                <mesh filename="package://sipder_robot/meshes/hip2.STL" />
+                <mesh filename="package://sipder_robot/meshes/spibot/hip2.STL" />
             </geometry>
             <material name="IndianRed">
@@ -261,5 +244,5 @@
             <origin xyz="0 0 0" rpy="0 0 0" />
             <geometry>
-                <mesh filename="package://sipder_robot/meshes/hip2.STL" />
+                <mesh filename="package://sipder_robot/meshes/spibot/hip2.STL" />
             </geometry>
         </collision>
@@ -281,5 +264,5 @@
             <origin xyz="0 0 0" rpy="0 0 0" />
             <geometry>
-                <mesh filename="package://sipder_robot/meshes/thigh2.STL" />
+                <mesh filename="package://sipder_robot/meshes/spibot/thigh2.STL" />
             </geometry>
             <material name="Green">
@@ -290,5 +273,5 @@
             <origin xyz="0 0 0" rpy="0 0 0" />
             <geometry>
-                <mesh filename="package://sipder_robot/meshes/thigh2.STL" />
+                <mesh filename="package://sipder_robot/meshes/spibot/thigh2.STL" />
             </geometry>
         </collision>
@@ -310,5 +293,5 @@
             <origin xyz="0 0 0" rpy="0 0 0" />
             <geometry>
-                <mesh filename="package://sipder_robot/meshes/shank2.STL" />
+                <mesh filename="package://sipder_robot/meshes/spibot/shank2.STL" />
             </geometry>
             <material name="Cyan">
@@ -319,5 +302,5 @@
             <origin xyz="0 0 0" rpy="0 0 0" />
             <geometry>
-                <mesh filename="package://sipder_robot/meshes/shank2.STL" />
+                <mesh filename="package://sipder_robot/meshes/spibot/shank2.STL" />
             </geometry>
         </collision>
@@ -362,5 +345,5 @@
             <origin xyz="0 0 0" rpy="0 0 0" />
             <geometry>
-                <mesh filename="package://sipder_robot/meshes/foot2.STL" />
+                <mesh filename="package://sipder_robot/meshes/spibot/foot2.STL" />
             </geometry>
             <material name="SkyBlue">
@@ -371,5 +354,5 @@
             <origin xyz="0 0 0" rpy="0 0 0" />
             <geometry>
-                <mesh filename="package://sipder_robot/meshes/foot2.STL" />
+                <mesh filename="package://sipder_robot/meshes/spibot/foot2.STL" />
             </geometry>
         </collision>
@@ -384,5 +367,5 @@
             <origin xyz="0 0 0" rpy="0 0 0" />
             <geometry>
-                <mesh filename="package://sipder_robot/meshes/hip3.STL" />
+                <mesh filename="package://sipder_robot/meshes/spibot/hip3.STL" />
             </geometry>
             <material name="IndianRed">
@@ -393,5 +376,5 @@
             <origin xyz="0 0 0" rpy="0 0 0" />
             <geometry>
-                <mesh filename="package://sipder_robot/meshes/hip3.STL" />
+                <mesh filename="package://sipder_robot/meshes/spibot/hip3.STL" />
             </geometry>
         </collision>
@@ -413,5 +396,5 @@
             <origin xyz="0 0 0" rpy="0 0 0" />
             <geometry>
-                <mesh filename="package://sipder_robot/meshes/thigh3.STL" />
+                <mesh filename="package://sipder_robot/meshes/spibot/thigh3.STL" />
             </geometry>
             <material name="Green">
@@ -422,5 +405,5 @@
             <origin xyz="0 0 0" rpy="0 0 0" />
             <geometry>
-                <mesh filename="package://sipder_robot/meshes/thigh3.STL" />
+                <mesh filename="package://sipder_robot/meshes/spibot/thigh3.STL" />
             </geometry>
         </collision>
@@ -442,5 +425,5 @@
             <origin xyz="0 0 0" rpy="0 0 0" />
             <geometry>
-                <mesh filename="package://sipder_robot/meshes/shank3.STL" />
+                <mesh filename="package://sipder_robot/meshes/spibot/shank3.STL" />
             </geometry>
             <material name="Cyan">
@@ -451,5 +434,5 @@
             <origin xyz="0 0 0" rpy="0 0 0" />
             <geometry>
-                <mesh filename="package://sipder_robot/meshes/shank3.STL" />
+                <mesh filename="package://sipder_robot/meshes/spibot/shank3.STL" />
             </geometry>
         </collision>
@@ -494,5 +477,5 @@
             <origin xyz="0 0 0" rpy="0 0 0" />
             <geometry>
-                <mesh filename="package://sipder_robot/meshes/foot3.STL" />
+                <mesh filename="package://sipder_robot/meshes/spibot/foot3.STL" />
             </geometry>
             <material name="SkyBlue">
@@ -503,5 +486,5 @@
             <origin xyz="0 0 0" rpy="0 0 0" />
             <geometry>
-                <mesh filename="package://sipder_robot/meshes/foot3.STL" />
+                <mesh filename="package://sipder_robot/meshes/spibot/foot3.STL" />
             </geometry>
         </collision>
@@ -516,5 +499,5 @@
             <origin xyz="0 0 0" rpy="0 0 0" />
             <geometry>
-                <mesh filename="package://sipder_robot/meshes/hip4.STL" />
+                <mesh filename="package://sipder_robot/meshes/spibot/hip4.STL" />
             </geometry>
             <material name="IndianRed">
@@ -525,5 +508,5 @@
             <origin xyz="0 0 0" rpy="0 0 0" />
             <geometry>
-                <mesh filename="package://sipder_robot/meshes/hip4.STL" />
+                <mesh filename="package://sipder_robot/meshes/spibot/hip4.STL" />
             </geometry>
         </collision>
@@ -545,5 +528,5 @@
             <origin xyz="0 0 0" rpy="0 0 0" />
             <geometry>
-                <mesh filename="package://sipder_robot/meshes/thigh4.STL" />
+                <mesh filename="package://sipder_robot/meshes/spibot/thigh4.STL" />
             </geometry>
             <material name="Green">
@@ -554,5 +537,5 @@
             <origin xyz="0 0 0" rpy="0 0 0" />
             <geometry>
-                <mesh filename="package://sipder_robot/meshes/thigh4.STL" />
+                <mesh filename="package://sipder_robot/meshes/spibot/thigh4.STL" />
             </geometry>
         </collision>
@@ -574,5 +557,5 @@
             <origin xyz="0 0 0" rpy="0 0 0" />
             <geometry>
-                <mesh filename="package://sipder_robot/meshes/shank4.STL" />
+                <mesh filename="package://sipder_robot/meshes/spibot/shank4.STL" />
             </geometry>
             <material name="Cyan">
@@ -583,5 +566,5 @@
             <origin xyz="0 0 0" rpy="0 0 0" />
             <geometry>
-                <mesh filename="package://sipder_robot/meshes/shank4.STL" />
+                <mesh filename="package://sipder_robot/meshes/spibot/shank4.STL" />
             </geometry>
         </collision>
@@ -626,5 +609,5 @@
             <origin xyz="0 0 0" rpy="0 0 0" />
             <geometry>
-                <mesh filename="package://sipder_robot/meshes/foot4.STL" />
+                <mesh filename="package://sipder_robot/meshes/spibot/foot4.STL" />
             </geometry>
             <material name="SkyBlue">
@@ -635,5 +618,5 @@
             <origin xyz="0 0 0" rpy="0 0 0" />
             <geometry>
-                <mesh filename="package://sipder_robot/meshes/foot4.STL" />
+                <mesh filename="package://sipder_robot/meshes/spibot/foot4.STL" />
             </geometry>
         </collision>
