Commit message: 将叶片加载在环境中，改变机器人原始位置

File: src/sipder_robot/urdf/WindTurbine_Blade.urdf (robot description, URDF)
Before this commit: robot WindTurbine_Blade, 1 links, 0 joints
Links:
- removed link base_link
- added link Wind_Turbine, mass 0; collision mesh filename=package://sipder_robot/meshes/spibot/Wind_Turbine.STL; visual mesh filename=package://sipder_robot/meshes/spibot/Wind_Turbine.STL

File: src/sipder_robot/xacro/gazebo/foot_add_grippers.xacro (robot description, xacro)
@@ -7,5 +7,5 @@
             <origin rpy="0 0 0" xyz="0 0 0"/>
             <geometry>
-                <cylinder length="0.005" radius="0.05" />
+                <cylinder radius="0.05" length="0.01"/>
             </geometry>
             <material name="transparent">
@@ -23,5 +23,5 @@
         <parent link="foot1" />
         <child link="vacuum_gripper1" />
-        <origin rpy="0 0 0" xyz="0 0 0" />
+        <origin rpy="0 0 0" xyz="0 0 0.052" />
         <limit effort="50" velocity="50" lower="0" upper="0" />
         <dynamics damping="0.0" friction="10"/>
@@ -41,5 +41,5 @@
             <origin rpy="0 0 0" xyz="0 0 0"/>
             <geometry>
-                <cylinder length="0.005" radius="0.05" />
+                <cylinder radius="0.05" length="0.01"/>
             </geometry>
             <material name="transparent">
@@ -57,5 +57,5 @@
         <parent link="foot2" />
         <child link="vacuum_gripper2" />
-        <origin rpy="0 0 0" xyz="0 0 0" />
+        <origin rpy="0 0 0" xyz="0 0 0.052" />
         <limit effort="50" velocity="50" lower="0" upper="0" />
         <dynamics damping="0.0" friction="10"/>
@@ -75,5 +75,5 @@
             <origin rpy="0 0 0" xyz="0 0 0"/>
             <geometry>
-                <cylinder length="0.005" radius="0.05" />
+                <cylinder radius="0.05" length="0.01"/>
             </geometry>
             <material name="transparent">
@@ -91,5 +91,5 @@
         <parent link="foot3" />
         <child link="vacuum_gripper3" />
-        <origin rpy="0 0 0" xyz="0 0 0" />
+        <origin rpy="0 0 0" xyz="0 0 0.052" />
         <limit effort="50" velocity="50" lower="0" upper="0" />
         <dynamics damping="0.0" friction="10"/>
@@ -109,5 +109,5 @@
             <origin rpy="0 0 0" xyz="0 0 0"/>
             <geometry>
-                <cylinder length="0.005" radius="0.05" />
+                <cylinder radius="0.05" length="0.01"/>
             </geometry>
             <material name="transparent">
@@ -125,5 +125,5 @@
         <parent link="foot4" />
         <child link="vacuum_gripper4" />
-        <origin rpy="0 0 0" xyz="0 0 0" />
+        <origin rpy="0 0 0" xyz="0 0 0.052" />
         <limit effort="50" velocity="50" lower="0" upper="0" />
         <dynamics damping="0.0" friction="10"/>
@@ -139,2 +139,142 @@
     </gazebo>
 </robot>
+<!-- <?xml version="1.0"?>
+<robot name="my_grippers"
+    xmlns:xacro="http://www.ros.org/wiki/xacro">
+    <link name="vacuum_gripper1">
+        <gravity>0</gravity>
+        <visual>
+            <origin rpy="0 0 0" xyz="0 0 0"/>
+            <geometry>
+                <cylinder length="0.005" radius="0.05" />
+            </geometry>
+            <material name="transparent">
+                <color rgba="0 0 0 0"/>
+            </material>
+        </visual>
+        <inertial>
+            <origin rpy="0 0 0" xyz="0.000000 0.000000 0.000000"/>
+            <mass value="0.0001"/>
+            <inertia ixx="1e-08" ixy="0" ixz="0" iyy="1e-08" iyz="0" izz="1e-08"/>
+        </inertial>
+    </link>
+    <joint name="gripper1_joint" type="revolute">
+        <axis xyz="1 0 0" />
+        <parent link="foot1" />
+        <child link="vacuum_gripper1" />
+        <origin rpy="0 0 0" xyz="0 0 0" />
+        <limit effort="50" velocity="50" lower="0" upper="0" />
+        <dynamics damping="0.0" friction="10"/>
+    </joint>
+    <gazebo reference="vacuum_gripper1">
+        <mu1>500</mu1>
+        <mu2>500</mu2>
+        <minDepth>0.003</minDepth>
+        <maxVel>0</maxVel>
+        <kp>1000000.0</kp>
+        <kd>1.0</kd>
+        <material>Gazebo/Grey</material>
+    </gazebo>
+    <link name="vacuum_gripper2">
+        <gravity>0</gravity>
+        <visual>
+            <origin rpy="0 0 0" xyz="0 0 0"/>
+            <geometry>
+                <cylinder length="0.005" radius="0.05" />
+            </geometry>
+            <material name="transparent">
+                <color rgba="0 0 0 0"/>
+            </material>
+        </visual>
+        <inertial>
+            <origin rpy="0 0 0" xyz="0.000000 0.000000 0.000000"/>
+            <mass value="0.0001"/>
+            <inertia ixx="1e-08" ixy="0" ixz="0" iyy="1e-08" iyz="0" izz="1e-08"/>
+        </inertial>
+    </link>
+    <joint name="gripper2_joint" type="revolute">
+        <axis xyz="1 0 0" />
+        <parent link="foot2" />
+        <child link="vacuum_gripper2" />
+        <origin rpy="0 0 0" xyz="0 0 0" />
+        <limit effort="50" velocity="50" lower="0" upper="0" />
+        <dynamics damping="0.0" friction="10"/>
+    </joint>
+    <gazebo reference="vacuum_gripper2">
+        <mu1>500</mu1>
+        <mu2>500</mu2>
+        <minDepth>0.003</minDepth>
+        <maxVel>0</maxVel>
+        <kp>1000000.0</kp>
+        <kd>1.0</kd>
+        <material>Gazebo/Grey</material>
+    </gazebo>
+    <link name="vacuum_gripper3">
+        <gravity>0</gravity>
+        <visual>
+            <origin rpy="0 0 0" xyz="0 0 0"/>
+            <geometry>
+                <cylinder length="0.005" radius="0.05" />
+            </geometry>
+            <material name="transparent">
+                <color rgba="0 0 0 0"/>
+            </material>
+        </visual>
+        <inertial>
+            <origin rpy="0 0 0" xyz="0.000000 0.000000 0.000000"/>
+            <mass value="0.0001"/>
+            <inertia ixx="1e-08" ixy="0" ixz="0" iyy="1e-08" iyz="0" izz="1e-08"/>
+        </inertial>
+    </link>
+    <joint name="gripper3_joint" type="revolute">
+        <axis xyz="1 0 0" />
+        <parent link="foot3" />
+        <child link="vacuum_gripper3" />
+        <origin rpy="0 0 0" xyz="0 0 0" />
+        <limit effort="50" velocity="50" lower="0" upper="0" />
+        <dynamics damping="0.0" friction="10"/>
+    </joint>
+    <gazebo reference="vacuum_gripper3">
+        <mu1>500</mu1>
+        <mu2>500</mu2>
+        <minDepth>0.003</minDepth>
+        <maxVel>0</maxVel>
+        <kp>1000000.0</kp>
+        <kd>1.0</kd>
+        <material>Gazebo/Grey</material>
+    </gazebo>
+    <link name="vacuum_gripper4">
+        <gravity>0</gravity>
+        <visual>
+            <origin rpy="0 0 0" xyz="0 0 0"/>
+            <geometry>
+                <cylinder length="0.005" radius="0.05" />
+            </geometry>
+            <material name="transparent">
+                <color rgba="0 0 0 0"/>
+            </material>
+        </visual>
+        <inertial>
+            <origin rpy="0 0 0" xyz="0.000000 0.000000 0.000000"/>
+            <mass value="0.0001"/>
+            <inertia ixx="1e-08" ixy="0" ixz="0" iyy="1e-08" iyz="0" izz="1e-08"/>
+        </inertial>
+    </link>
+    <joint name="gripper4_joint" type="revolute">
+        <axis xyz="1 0 0" />
+        <parent link="foot4" />
+        <child link="vacuum_gripper4" />
+        <origin rpy="0 0 0" xyz="0 0 0" />
+        <limit effort="50" velocity="50" lower="0" upper="0" />
+        <dynamics damping="0.0" friction="10"/>
+    </joint>
+    <gazebo reference="vacuum_gripper4">
+        <mu1>500</mu1>
+        <mu2>500</mu2>
+        <minDepth>0.003</minDepth>
+        <maxVel>0</maxVel>
+        <kp>1000000.0</kp>
+        <kd>1.0</kd>
+        <material>Gazebo/Grey</material>
+    </gazebo>
+</robot> -->

File: src/sipder_robot/xacro/spibot.xacro (robot description, xacro)
@@ -29,5 +29,5 @@
     </link>
     <joint name="dummy_joint" type="fixed">
-        <origin rpy="0 0 0" xyz="0 0 0"/>
+        <origin rpy="0 0 0" xyz="-2.0 -2.0 0.3"/>
         <parent link="dummy"/>
         <child link="base_link"/>
