Commit message: 20250326

File: src/sipder_robot/xacro/gazebo/laser.xacro (robot description, xacro)
@@ -1,35 +1,33 @@
-<?xml version="1.0"?>
-<robot name="my_sensors" xmlns:xacro="http://wiki.ros.org/xacro">
 <?xml version="1.0"?>
 <robot name="my_sensors" xmlns:xacro="http://wiki.ros.org/xacro">
   <!-- 雷达 -->
-  <gazebo reference="lidar">                  <!--  修改成自己雷达的名字 -->
-    <sensor type="ray" name="rplidar">        <!-- 设置雷达类型 -->
+  <gazebo reference="lidar">
+    <sensor type="ray" name="rplidar">
       <pose>0 0 0 0 0 0</pose>
       <visualize>true</visualize>
-      <update_rate>5</update_rate>              <!-- 雷达更新频率 -->
+      <update_rate>5.5</update_rate>
       <ray>
         <scan>
           <horizontal>
-            <samples>360</samples>                         <!-- 旋转一周所发出的射线 -->
-            <resolution>1</resolution>      <!-- 分辨率，每n个射线有一个测距，降低仿真环境压力 -->
-            <min_angle>-3.14</min_angle>     <!-- 雷达采样范围 ，向左转3个弧度 -->
-            <max_angle>3.14</max_angle>       <!-- 雷达采样范围 ，向右转3个弧度  -->
+            <samples>360</samples>
+            <resolution>1</resolution>
+            <min_angle>-3.14</min_angle>
+            <max_angle>3.14</max_angle>
           </horizontal>
         </scan>
         <range>
-          <min>0.10</min>                   <!-- 采样距离小于0.1，采集不到 -->
-          <max>30.0</max>                    <!-- 大于30m，采样不到 -->
-          <resolution>0.01</resolution>       <!-- 精度，最多精确到1厘米 -->
+          <min>0.5</min>
+          <max>100.0</max>
+          <resolution>0.01</resolution>
         </range>
-        <noise>                            <!-- 增强仿真 -->
-          <type>gaussian</type>             <!-- 高斯噪音 -->
-          <mean>0.0</mean>                  <!-- 平均值 -->
-          <stddev>0.01</stddev>             <!-- 标准差 -->
+        <noise>
+          <type>gaussian</type>
+          <mean>0.0</mean>
+          <stddev>0.01</stddev>
         </noise>
       </ray>
       <plugin name="gazebo_rplidar" filename="libgazebo_ros_laser.so">
-        <topicName>/spibot_gazebo/laser_scan</topicName>               <!-- 注意话题，需要订阅 -->
-        <frameName>lidar</frameName>               <!-- 与自己雷达传感器名字相同 -->
+        <topicName>/scan</topicName>
+        <frameName>lidar</frameName>
       </plugin>
     </sensor>

File: src/sipder_robot/xacro/spibot.xacro (robot description, xacro)
@@ -28,9 +28,18 @@
         </visual>
     </link>
-    <joint name="dummy_joint" type="fixed">
-        <origin rpy="0 0 0" xyz="-2.0 -2.0 0.3"/>
-        <parent link="dummy"/>
-        <child link="base_link"/>
-    </joint>
+    <xacro:if value="$(arg ADD_WIND_TURBINE)">
+        <joint name="dummy_joint" type="fixed">
+            <origin rpy="1.57 0 0" xyz="0.05 -1.05 8.0"/>
+            <parent link="dummy"/>
+            <child link="base_link"/>
+        </joint>
+    </xacro:if>
+    <xacro:unless value="$(arg ADD_WIND_TURBINE)">
+        <joint name="dummy_joint" type="fixed">
+            <origin rpy="0 0 0" xyz="0.0 0.0 0.0"/>
+            <parent link="dummy"/>
+            <child link="base_link"/>
+        </joint>
+    </xacro:unless>
     <link name="base_link">
         <inertial>

File: src/sipder_robot/xacro/spibot_with_sensors.xacro (robot description, xacro)
@@ -7,6 +7,6 @@
     <xacro:include filename="gazebo/kinect.xacro"/>
     <!-- 给机器人的lidar增加三维激光雷达以生成点云数据，laser雷达是生成二维点云数据，二者选其一 -->
-    <xacro:include filename="$(find sipder_robot)/xacro/gazebo/velodyne.xacro"/>
-    <!-- <xacro:include filename="$(find sipder_robot)/xacro/gazebo/laser.xacro"/> -->
+    <!-- <xacro:include filename="$(find sipder_robot)/xacro/gazebo/velodyne.xacro"/> -->
+    <xacro:include filename="$(find sipder_robot)/xacro/gazebo/laser.xacro"/>
     <!-- 给机器人的camera增加imu以显示自身状态 -->
     <xacro:include filename="gazebo/imu.xacro"/>
